File: SNES_RGB_BYPASS_AMP.kicad_pcb (KiCad board)
At the start: 2 copper layers, 16 x 29.5 mm, 16 parts, among them J1 RGB_Input, J2 SNES Multiout, U1 THS7374

Commit message: Update silkscreen
Other:
- board text added: "CS R G B"
Changed lines of the file:
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@@
     (property "ki_keywords" "cap capacitor")
     (attr smd)
-    (fp_text reference "C1" (at 2.3244 0.278 -180) (layer "F.SilkS")
-        (effects (font (size 1 1) (thickness 0.15)))
+    (fp_text reference "C1" (at 2.3244 0.278 180) (layer "F.SilkS")
+        (effects (font (size 0.8 0.8) (thickness 0.15)))
     )
     (fp_text value "1uF" (at 0 1.68 90) (layer "F.Fab")
@@
     (property "ki_keywords" "R res resistor")
     (attr smd)
-    (fp_text reference "R5" (at 2.5808 -0.2248 -180) (layer "F.SilkS")
-        (effects (font (size 1 1) (thickness 0.15)))
+    (fp_text reference "R5" (at 2.0808 -0.2248 180) (layer "F.SilkS")
+        (effects (font (size 0.8 0.8) (thickness 0.15)))
     )
     (fp_text value "75" (at 0 1.68 90) (layer "F.Fab")
@@
     (attr smd)
     (fp_text reference "R4" (at 0 1.5 90) (layer "F.SilkS")
-        (effects (font (size 1 1) (thickness 0.15)))
+        (effects (font (size 0.8 0.8) (thickness 0.15)))
     )
     (fp_text value "10K" (at 0 1.68 90) (layer "F.Fab")
@@
     (attr smd)
     (fp_text reference "R3" (at -2.5 0 180) (layer "F.SilkS")
-        (effects (font (size 1 1) (thickness 0.15)))
+        (effects (font (size 0.8 0.8) (thickness 0.15)))
     )
     (fp_text value "750" (at 0 1.68 90) (layer "F.Fab")
@@
         (effects (font (size 1 1) (thickness 0.15)))
     )
-    (fp_line (start -1.33 1.27) (end -1.33 8.95)
-      (stroke (width 0.12) (type solid)) (layer "F.SilkS"))
-    (fp_line (start -1.33 1.27) (end 1.33 1.27)
-      (stroke (width 0.12) (type solid)) (layer "F.SilkS"))
-    (fp_line (start -1.33 8.95) (end 1.33 8.95)
-      (stroke (width 0.12) (type solid)) (layer "F.SilkS"))
-    (fp_line (start 0 -1.33) (end 1.33 -1.33)
-      (stroke (width 0.12) (type solid)) (layer "F.SilkS"))
-    (fp_line (start 1.33 -1.33) (end 1.33 0)
-      (stroke (width 0.12) (type solid)) (layer "F.SilkS"))
-    (fp_line (start 1.33 1.27) (end 1.33 8.95)
-      (stroke (width 0.12) (type solid)) (layer "F.SilkS"))
     (fp_line (start -1.8 -1.8) (end 1.75 -1.8)
       (stroke (width 0.05) (type solid)) (layer "F.CrtYd"))
@@
     (fp_line (start 1.75 9.4) (end -1.8 9.4)
       (stroke (width 0.05) (type solid)) (layer "F.CrtYd"))
-    (fp_line (start -1.27 -1.27) (end 0.635 -1.27)
-      (stroke (width 0.1) (type solid)) (layer "F.Fab"))
-    (fp_line (start -1.27 8.89) (end -1.27 -1.27)
-      (stroke (width 0.1) (type solid)) (layer "F.Fab"))
-    (fp_line (start 0.635 -1.27) (end 1.27 -0.635)
-      (stroke (width 0.1) (type solid)) (layer "F.Fab"))
-    (fp_line (start 1.27 -0.635) (end 1.27 8.89)
-      (stroke (width 0.1) (type solid)) (layer "F.Fab"))
-    (fp_line (start 1.27 8.89) (end -1.27 8.89)
-      (stroke (width 0.1) (type solid)) (layer "F.Fab"))
     (pad "1" smd rect (at 0 0 90) (size 2 2) (layers "F.Cu" "F.Paste" "F.Mask")
       (net 3 "/CSync") (pinfunction "Pin_1") (pintype "passive"))
@@
     (attr smd)
     (fp_text reference "R2" (at -2.5 0 180) (layer "F.SilkS")
-        (effects (font (size 1 1) (thickness 0.15)))
+        (effects (font (size 0.8 0.8) (thickness 0.15)))
     )
     (fp_text value "750" (at 0 1.68 90) (layer "F.Fab")
@@
     (property "ki_keywords" "R res resistor")
     (attr smd)
-    (fp_text reference "R7" (at 2.5808 -0.2224 -180) (layer "F.SilkS")
-        (effects (font (size 1 1) (thickness 0.15)))
+    (fp_text reference "R7" (at 2.0808 -0.2224 180) (layer "F.SilkS")
+        (effects (font (size 0.8 0.8) (thickness 0.15)))
     )
     (fp_text value "75" (at 0 1.68 90) (layer "F.Fab")
@@
     (property "ki_keywords" "R res resistor")
     (attr smd)
-    (fp_text reference "R8" (at 2.5808 0.0264 -180) (layer "F.SilkS")
-        (effects (font (size 1 1) (thickness 0.15)))
+    (fp_text reference "R8" (at 2.0808 0.5264 180) (layer "F.SilkS")
+        (effects (font (size 0.8 0.8) (thickness 0.15)))
     )
     (fp_text value "75" (at 0 1.68 90) (layer "F.Fab")
@@
     (attr smd)
     (fp_text reference "R1" (at -2.5 0 180) (layer "F.SilkS")
-        (effects (font (size 1 1) (thickness 0.15)))
+        (effects (font (size 0.8 0.8) (thickness 0.15)))
     )
     (fp_text value "750" (at 0 1.68 90) (layer "F.Fab")
@@
     (property "ki_keywords" "R res resistor")
     (attr smd)
-    (fp_text reference "R6" (at 2.6164 -0.1236 -180) (layer "F.SilkS")
-        (effects (font (size 1 1) (thickness 0.15)))
+    (fp_text reference "R6" (at 2.1164 -0.1236 180) (layer "F.SilkS")
+        (effects (font (size 0.8 0.8) (thickness 0.15)))
     )
     (fp_text value "75" (at 0 1.68 90) (layer "F.Fab")
@@
     (property "ki_keywords" "cap capacitor")
     (attr smd)
-    (fp_text reference "C2" (at 2.3752 -0.2422 -180) (layer "F.SilkS")
-        (effects (font (size 1 1) (thickness 0.15)))
+    (fp_text reference "C2" (at 2.3752 -0.2422 180) (layer "F.SilkS")
+        (effects (font (size 0.8 0.8) (thickness 0.15)))
     )
     (fp_text value "0.1uF" (at 0 1.68 90) (layer "F.Fab")
@@
   (gr_line (start 127.5 77) (end 127.5 99)
     (stroke (width 0.1) (type default)) (layer "Edge.Cuts"))
-  (gr_text "TTL" (at 134 86.5) (layer "F.SilkS")
-    (effects (font (size 0.8 0.8) (thickness 0.1) bold) (justify left bottom))
+  (gr_text "CS  R   G   B" (at 132.5 96.5) (layer "F.SilkS")
+    (effects (font (size 0.8 0.8) (thickness 0.15)) (justify left bottom))
+  )
+  (gr_text "TTL" (at 134 87) (layer "F.SilkS")
+    (effects (font (size 0.8 0.8) (thickness 0.15) bold) (justify left bottom))
   )
   (gr_text "ON" (at 129 91 90) (layer "F.SilkS")
-    (effects (font (size 0.8 0.8) (thickness 0.1) bold) (justify left bottom))
+    (effects (font (size 0.8 0.8) (thickness 0.15) bold) (justify left bottom))
   )
   (gr_text "LPF" (at 133 93 90) (layer "F.SilkS")
-    (effects (font (size 1 1) (thickness 0.15)) (justify left bottom))
+    (effects (font (size 0.8 0.8) (thickness 0.15)) (justify left bottom))
   )
   (gr_text "OFF" (at 129 94.5 90) (layer "F.SilkS")
-    (effects (font (size 0.8 0.8) (thickness 0.1) bold) (justify left bottom))
+    (effects (font (size 0.8 0.8) (thickness 0.15) bold) (justify left bottom))
   )
   (segment (start 131.1656 70.871) (end 129.9906 72.046) (width 0.25) (layer "F.Cu") (net 1))

Commit message: fix errors
Parts:
- J1: value RGB_Input -> INPUT; footprint Connector_PinSocket_2.54mm:PinSocket_1x04_P2.54mm_Vertical -> Connector_PinHeader_2.54mm:PinHeader_1x04_P2.54mm_Vertical
- moved R4 12.9 mm to (129.3, 84.1), turned to 90 degrees
- moved R8 6.56 mm to (141.5, 78.5)
- moved C1 5.13 mm to (132.3, 80.5), turned to 90 degrees
- moved JP2 4.25 mm to (130.2, 89.2), turned to 90 degrees
- moved R6 4.03 mm to (137.5, 78.5)
- moved R5 3.88 mm to (135.5, 78.5)
- moved JP1 3.19 mm to (133.1, 89.2)
- moved R7 1.60 mm to (139.5, 78.5)
Connections:
- J1 pad 2: /R -> /B
- J1 pad 4: /B -> /R
- J2 pad 3: unconnected-(J2-Pin_3-Pad3) -> /CSync'
- J2 pad 6: unconnected-(J2-Pin_6-Pad6) -> GND
- J2 pad 8: /CSync' -> unconnected-(J2-Pin_8-Pad8)
- R1 pad 2: /B -> /R
- R3 pad 2: /R -> /B
- R6 pad 1: /R' -> /B'
- R8 pad 1: /B' -> /R'
- U1 pad 2: /R -> /B
- U1 pad 4: /B -> /R
Routing:
- net VCC: track 47.2 -> 27.4 mm, vias 4 -> 2
- net Net-(JP1-B): track 20.7 -> 14.6 mm, vias 2 -> 0
- net Net-(JP3-A): track 12.6 -> 7.65 mm, vias 2 -> 0
- net GND: track 51.8 -> 47.3 mm, vias 9 -> 6
- net /G': track 6.86 -> 11.2 mm
- net Net-(U1-CH2_OUT): track 7.66 -> 3.40 mm, vias 2 -> 0
- net Net-(U1-CH4_OUT): track 8.21 -> 3.99 mm, vias 2 -> 0
- net /CSync': track 14.6 -> 12.0 mm
- net Net-(JP2-B): track 1.90 -> 4.45 mm
- net /R': track 3.04 -> 4.21 mm
- net /B': track 7.16 -> 8.18 mm
- net Net-(U1-CH3_OUT): track 4.33 -> 3.37 mm
- net /B: track 10.4 -> 11.0 mm
Other:
- board text added: "CS B G R"
- board text removed: "CS R G B"
