File: SNES_RGB_BYPASS_AMP.kicad_sch (KiCad schematic)
At the start: 16 parts, among them J1 RGB_Input, J2 SNES Multiout, U1 THS7374

Commit message: fix errors
Parts:
- removed J1: RGB_Input, Connector_PinSocket_2.54mm:PinSocket_1x04_P2.54mm_Vertical, symbol Connector:Conn_01x04_Pin
- added J1: INPUT, Connector_PinHeader_2.54mm:PinHeader_1x04_P2.54mm_Vertical, symbol Connector_Generic:Conn_01x04
Connections:
- net B: now also R3.2, U1.2 (CH2_IN), J1.2 (Pin_2); no longer R1.2, U1.4 (CH4_IN)
- net B': now also R6.1; no longer R8.1
- net CSync: now also J1.1 (Pin_1)
- net CSync': now also J2.3 (Pin_3); no longer J2.8 (Pin_8)
- net G: now also J1.3 (Pin_3)
- net GND: now also J2.6 (Pin_6)
- net R: now also R1.2, U1.4 (CH4_IN), J1.4 (Pin_4); no longer R3.2, U1.2 (CH2_IN)
- net R': now also R8.1; no longer R6.1
- no-connect marks 6 -> 5
Changed lines of the file:
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@@
   (junction (at 121.92 99.06) (diameter 0) (color 0 0 0 0)
   )
-  (no_connect (at 99.06 60.96))
+  (no_connect (at 86.36 66.04))
   (no_connect (at 99.06 66.04))
-  (no_connect (at 86.36 63.5))
   (no_connect (at 99.06 68.58))
   (no_connect (at 86.36 71.12))
@@
     (stroke (width 0) (type default))
   )
-  (label "CSync'" (at 86.36 66.04 180) (fields_autoplaced)
-    (effects (font (size 1.27 1.27)) (justify right bottom))
-  )
-  (label "B" (at 60.96 81.28 0) (fields_autoplaced)
+  (label "CSync'" (at 99.06 60.96 0) (fields_autoplaced)
+    (effects (font (size 1.27 1.27)) (justify left bottom))
+  )
+  (label "B" (at 60.96 76.2 0) (fields_autoplaced)
     (effects (font (size 1.27 1.27)) (justify left bottom))
   )
@@
     (effects (font (size 1.27 1.27)) (justify left bottom))
   )
-  (label "B'" (at 198.12 63.5 90) (fields_autoplaced)
+  (label "B'" (at 182.88 63.5 90) (fields_autoplaced)
     (effects (font (size 1.27 1.27)) (justify left bottom))
   )
@@
     (effects (font (size 1.27 1.27)) (justify left bottom))
   )
-  (label "R'" (at 182.88 63.5 90) (fields_autoplaced)
+  (label "R'" (at 198.12 63.5 90) (fields_autoplaced)
     (effects (font (size 1.27 1.27)) (justify left bottom))
   )
@@
     (effects (font (size 1.27 1.27)) (justify left bottom))
   )
-  (label "R" (at 93.98 99.06 0) (fields_autoplaced)
+  (label "R" (at 93.98 104.14 0) (fields_autoplaced)
     (effects (font (size 1.27 1.27)) (justify left bottom))
   )
@@
     (effects (font (size 1.27 1.27)) (justify left bottom))
   )
-  (label "R" (at 60.96 76.2 0) (fields_autoplaced)
+  (label "R" (at 60.96 81.28 0) (fields_autoplaced)
     (effects (font (size 1.27 1.27)) (justify left bottom))
   )
@@
     (effects (font (size 1.27 1.27)) (justify right bottom))
   )
-  (label "B" (at 93.98 104.14 0) (fields_autoplaced)
+  (label "B" (at 93.98 99.06 0) (fields_autoplaced)
     (effects (font (size 1.27 1.27)) (justify left bottom))
   )
@@
     )
   )
-  (symbol (lib_id "Connector:Conn_01x04_Pin") (at 50.8 76.2 0) (unit 1)
-    (in_bom yes) (on_board yes) (dnp no) (fields_autoplaced)
-    (property "Reference" "J1" (at 51.435 68.326 0)
-      (effects (font (size 1.27 1.27)))
-    )
-    (property "Value" "RGB_Input" (at 51.435 70.866 0)
-      (effects (font (size 1.27 1.27)))
-    )
-    (property "Footprint" "Connector_PinSocket_2.54mm:PinSocket_1x04_P2.54mm_Vertical" (at 50.8 76.2 0)
-      (effects (font (size 1.27 1.27)) hide)
-    )
-    (property "Datasheet" "~" (at 50.8 76.2 0)
-      (effects (font (size 1.27 1.27)) hide)
-    )
-    (pin "1")
-    (pin "2")
-    (pin "3")
-    (pin "4")
-    (instances
-      (project "SNES_RGB_BYPASS_AMP"
-        (path "/db7397df-a245-4004-bbf4-7c910e0e8a46"
-          (reference "J1") (unit 1)
-        )
-      )
-    )
-  )
   (symbol (lib_id "Device:R_US") (at 168.91 129.54 90) (unit 1)
     (in_bom yes) (on_board yes) (dnp no) (fields_autoplaced)
@@
         (path "/db7397df-a245-4004-bbf4-7c910e0e8a46"
           (reference "R5") (unit 1)
+        )
+      )
+    )
+  )
+  (symbol (lib_id "Connector_Generic:Conn_01x04") (at 50.8 76.2 0) (mirror y) (unit 1)
+    (in_bom yes) (on_board yes) (dnp no)
+    (property "Reference" "J1" (at 48.26 76.2 0)
+      (effects (font (size 1.27 1.27)) (justify left))
+    )
+    (property "Value" "INPUT" (at 48.26 78.74 0)
+      (effects (font (size 1.27 1.27)) (justify left))
+    )
+    (property "Footprint" "Connector_PinHeader_2.54mm:PinHeader_1x04_P2.54mm_Vertical" (at 50.8 76.2 0)
+      (effects (font (size 1.27 1.27)) hide)
+    )
+    (property "Datasheet" "~" (at 50.8 76.2 0)
+      (effects (font (size 1.27 1.27)) hide)
+    )
+    (pin "1")
+    (pin "2")
+    (pin "3")
+    (pin "4")
+    (instances
+      (project "SNES_RGB_BYPASS_AMP"
+        (path "/db7397df-a245-4004-bbf4-7c910e0e8a46"
+          (reference "J1") (unit 1)
         )
       )
@@
         )
       )
+    )
+  )
+  (symbol (lib_id "power:GND") (at 86.36 63.5 270) (unit 1)
+    (in_bom yes) (on_board yes) (dnp no) (fields_autoplaced)
+    (property "Reference" "#PWR09" (at 80.01 63.5 0)
+      (effects (font (size 1.27 1.27)) hide)
+    )
+    (property "Value" "GND" (at 82.55 63.5 90)
+      (effects (font (size 1.27 1.27)) (justify right))
+    )
+    (property "Footprint" "" (at 86.36 63.5 0)
+      (effects (font (size 1.27 1.27)) hide)
+    )
+    (property "Datasheet" "" (at 86.36 63.5 0)
+      (effects (font (size 1.27 1.27)) hide)
+    )
+    (pin "1")
+    (instances
+      (project "SNES_RGB_BYPASS_AMP"
+        (path "/db7397df-a245-4004-bbf4-7c910e0e8a46"
+          (reference "#PWR09") (unit 1)
+        )
+      )
